File: schematics/Falange/Falange.sch (EAGLE design)
At the start: 44 parts, among them IC1 7909, IC2 7809, IC3 TL082P

Commit message: update falange schematics
Connections:
- net N$1 renamed PWRTIP
- net N$3 renamed PWRSLV
Changed lines of the file:
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@@
 </segment>
 </net>
-<net name="N$1" class="0">
+<net name="PWRTIP" class="0">
 <segment>
 <pinref part="D1" gate="1" pin="C"/>
@@
 </segment>
 </net>
-<net name="N$3" class="0">
+<net name="PWRSLV" class="0">
 <segment>
 <pinref part="D3" gate="1" pin="A"/>
